File: parkir v1/PCB/Mega8.brd (EAGLE design)
At the start: 93 x 87 mm, 59 parts, among them IC1 ATMEGA8 (OR 168), IC2 DS1307, K1 ZF112, Q1 16000, T1 BC547, T2 BC557, T4 BC547

Commit message: relayout
Parts:
- removed C8: 100n, rcl:C050-025X075
- removed G1: B2430UNI, battery:B2430UNI
- removed IC2: DS1307, ds1307_pcf8583:DIL08
- removed LED0: A, led:LED3MM
- removed LED14: B, led:LED3MM
- removed Q2: (no value), crystal:TC26H
- removed R12, R13: 10k, rcl:0207/10
- added LED4: Q, led:LED3MM
- added LED5: Power, led:LED3MM
- LED1: value C -> A
- LED2: value TX -> B
- LED3: value Q -> C
- R19, R20, R21: value 10k -> 100k
- moved LED2 75.0 mm to (24.1, 81.3), turned to 90 degrees
- moved C5 63.5 mm to (78.7, 16.5), turned to 0 degrees
- moved DC1 61.6 mm to (76.8, 3.81)
- moved R3 44.5 mm to (35.6, 46.4)
- moved D2 41.0 mm to (45.7, 35.6), turned to 90 degrees
- moved R5 37.9 mm to (33.7, 26.0)
- moved R8 37.9 mm to (33.7, 28.6)
- moved T2 35.7 mm to (40.6, 28.6), turned to 90 degrees
- moved T1 35.2 mm to (48.9, 28.6), turned to 270 degrees
- moved C9 32.6 mm to (28.6, 16.5)
- moved D3 32.5 mm to (33.7, 21.0)
- moved R23 27.3 mm to (27.9, 34.3), turned to 180 degrees
- moved R10 25.6 mm to (45.7, 23.5), turned to 270 degrees
- moved R21 24.5 mm to (35.6, 62.9)
- moved R18 23.6 mm to (35.6, 48.9), turned to 180 degrees
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Connections:
- removed net N$10: IC1.28, IC2.6, R12.2
- removed net N$11: IC1.27, IC2.5, R13.2
- removed net N$12: C8.1, G1.+@4, IC2.3
- removed net N$24: IC2.1, Q2.2
- removed net N$25: IC2.2, Q2.1
- net +5V: now also R16.2; no longer IC2.8, R12.1, R13.1
- net GND: now also LED4.K, LED5.K; no longer C8.2, G1.-, G1.-@1, IC2.4, LED0.K, LED14.K
- net N$19: now also LED5.A; no longer LED2.A
- net N$21: now also LED4.A; no longer LED3.A
- net N$3: now also LED2.A; no longer LED14.A
- net N$30: now also K1.2; no longer K1.1, R16.2
- net N$32: now also LED3.A; no longer LED1.A
- net N$33: now also LED1.A; no longer LED0.A
- net N$4: now also K1.1; no longer K1.2
Routing:
- net GND: track 564.2 -> 433.6 mm
- net +5V: track 182.3 -> 120.4 mm
- net N$26: track 58.8 -> 25.8 mm
- net N$5: track 22.1 -> 53.9 mm
- net RLY: track 43.2 -> 11.4 mm
- net N$1: track 2.54 -> 33.4 mm
- net M8TXD: track 36.9 -> 9.52 mm
- net N$10: track 23.0 -> 0.00 mm
- net N$12: track 21.3 -> 0.00 mm
- net N$15: track 20.8 -> 41.3 mm
- net N$30: track 113.4 -> 97.1 mm, vias 2 -> 0
- net N$11: track 13.5 -> 0.00 mm
- net TX: track 69.7 -> 57.0 mm
- net RX: track 53.6 -> 41.0 mm
- net N$23: track 19.6 -> 32.2 mm
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Other:
- board size 93 x 87 mm -> 91.7 x 87 mm
